File: pcb/cpld-display.kicad_sch (KiCad schematic)
At the start: 18 parts, among them J1 USB_C_Receptacle_USB2.0_16P, J2 Conn_02x03_Odd_Even, U1 AMS1117-3.3, U2 AMS1117-1.8, U3 XC2C64A-7QFG48C

Commit message: Change jtag production properties
Parts:
- J2: now not fitted
Changed lines of the file:
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@@
 		(in_bom yes)
 		(on_board yes)
-		(dnp no)
+		(dnp yes)
 		(fields_autoplaced yes)
 		(property "Reference" "J2"

Commit message: Fix jtag tdo pin
Parts:
- removed C8: 100n, Capacitor_SMD:C_0402_1005Metric, symbol Device:C
Connections:
- net TDO: now reaches U3.40 (TDO)
- net TDO: now also J2.6 (Pin_6)
- no-connect marks 23 -> 21
Changed lines of the file:
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@@
 	)
 	(junction
-		(at 83.82 35.56)
-		(diameter 0)
-		(color 0 0 0 0)
-	)
-	(junction
-		(at 96.52 22.86)
-		(diameter 0)
-		(color 0 0 0 0)
-	)
-	(junction
 		(at 76.2 111.76)
 		(diameter 0)
@@
 	)
 	(no_connect
-		(at 111.76 33.02)
-	)
-	(no_connect
 		(at 45.72 109.22)
 	)
@@
 	)
 	(no_connect
-		(at 68.58 53.34)
-	)
-	(no_connect
 		(at 111.76 55.88)
 	)
@@
 	(wire
 		(pts
-			(xy 170.18 81.28) (xy 175.26 81.28)
+			(xy 63.5 53.34) (xy 68.58 53.34)
 		)
 		(stroke
@@
 	(wire
 		(pts
-			(xy 55.88 78.74) (xy 55.88 81.28)
+			(xy 170.18 81.28) (xy 175.26 81.28)
 		)
 		(stroke
@@
 	(wire
 		(pts
-			(xy 83.82 53.34) (xy 81.28 53.34)
+			(xy 55.88 78.74) (xy 55.88 81.28)
 		)
 		(stroke
@@
 	(wire
 		(pts
-			(xy 106.68 88.9) (xy 111.76 88.9)
+			(xy 83.82 53.34) (xy 81.28 53.34)
 		)
 		(stroke
@@
 	(wire
 		(pts
-			(xy 154.94 33.02) (xy 142.24 33.02)
+			(xy 106.68 88.9) (xy 111.76 88.9)
 		)
 		(stroke
@@
 	(wire
 		(pts
-			(xy 50.8 83.82) (xy 50.8 81.28)
+			(xy 154.94 33.02) (xy 142.24 33.02)
 		)
 		(stroke
@@
 	(wire
 		(pts
-			(xy 76.2 78.74) (xy 76.2 81.28)
+			(xy 50.8 83.82) (xy 50.8 81.28)
 		)
 		(stroke
@@
 	(wire
 		(pts
-			(xy 83.82 35.56) (xy 96.52 35.56)
+			(xy 76.2 78.74) (xy 76.2 81.28)
 		)
 		(stroke
@@
 	(wire
 		(pts
-			(xy 96.52 25.4) (xy 96.52 22.86)
-		)
-		(stroke
-			(width 0)
-			(type default)
-		)
-	)
-	(wire
-		(pts
 			(xy 121.92 22.86) (xy 121.92 25.4)
 		)
@@
 	(wire
 		(pts
-			(xy 96.52 22.86) (xy 83.82 22.86)
-		)
-		(stroke
-			(width 0)
-			(type default)
-		)
-	)
-	(wire
-		(pts
 			(xy 105.41 73.66) (xy 111.76 73.66)
 		)
@@
 	(wire
 		(pts
-			(xy 96.52 35.56) (xy 96.52 33.02)
-		)
-		(stroke
-			(width 0)
-			(type default)
-		)
-	)
-	(wire
-		(pts
 			(xy 129.54 93.98) (xy 129.54 96.52)
 		)
@@
 	(wire
 		(pts
+			(xy 106.68 33.02) (xy 111.76 33.02)
+		)
+		(stroke
+			(width 0)
+			(type default)
+		)
+	)
+	(wire
+		(pts
 			(xy 83.82 22.86) (xy 83.82 25.4)
 		)
@@
 	(wire
 		(pts
-			(xy 96.52 22.86) (xy 121.92 22.86)
+			(xy 83.82 22.86) (xy 121.92 22.86)
 		)
 		(stroke
@@
 		)
 	)
+	(label "TDO"
+		(at 63.5 53.34 0)
+		(fields_autoplaced yes)
+		(effects
+			(font
+				(size 1.27 1.27)
+			)
+			(justify left bottom)
+		)
+	)
 	(label "IN2A"
 		(at 170.18 50.8 0)
@@
 		)
 	)
+	(label "TDO"
+		(at 106.68 33.02 0)
+		(fields_autoplaced yes)
+		(effects
+			(font
+				(size 1.27 1.27)
+			)
+			(justify left bottom)
+		)
+	)
 	(label "IN2D"
 		(at 170.18 58.42 0)
@@
 					(unit 1)
 				)
-			)
-		)
-	)
-	(symbol
-		(lib_id "Device:C")
-		(at 96.52 29.21 0)
-		(unit 1)
-		(exclude_from_sim no)
-		(in_bom yes)
-		(on_board yes)
-		(dnp no)
-		(fields_autoplaced yes)
-		(property "Reference" "C8"
-			(at 100.33 27.9399 0)
-			(effects
-				(font
-					(size 1.27 1.27)
-				)
-				(justify left)
-			)
-		)
-		(property "Value" "100n"
-			(at 100.33 30.4799 0)
-			(effects
-				(font
-					(size 1.27 1.27)
-				)
-				(justify left)
-			)
-		)
-		(property "Footprint" "Capacitor_SMD:C_0402_1005Metric"
-			(at 97.4852 33.02 0)
-			(effects
-				(font
-					(size 1.27 1.27)
-				)
-				(hide yes)
-			)
-		)
-		(property "Datasheet" "~"
-			(at 96.52 29.21 0)
-			(effects
-				(font
-					(size 1.27 1.27)
-				)
-				(hide yes)
-			)
-		)
-		(property "Description" "Unpolarized capacitor"
-			(at 96.52 29.21 0)
-			(effects
-				(font
-					(size 1.27 1.27)
-				)
-				(hide yes)
-			)
-		)
-		(property "LCSC" "C1525"
-			(at 96.52 29.21 0)
-			(effects
-				(font
-					(size 1.27 1.27)
-				)
-				(hide yes)
-			)
-		)
-		(pin "1"
-		)
-		(pin "2"
-		)
-		(instances
-			(project "cpld-display"
-				(path "/b91428f0-b0b0-40b6-a29d-063fba957930"
-					(reference "C8")
-					(unit 1)
-				)
